File: electronic/pdu-board/pdu-board.kicad_pcb (KiCad board)
At the start: 2 copper layers, 400 x 30 mm, 38 parts, among them J1 Raspberry_D, J10 TERM, J11 SWITCH, J12 Raspberry_MGMT, J13 PWM_RPI, J14 FAN_B, J15 FAN_A, J2 Raspberry_C, J3 Raspberry_B, J4 Raspberry_A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

Commit message: RTC + GSM board
Parts:
- removed C1, C2, C3, C4: 100uF, Capacitor_THT:CP_Radial_D6.3mm_P2.50mm
- removed D1, D2, D3, D4: 1N4007, Diode_THT:D_DO-41_SOD81_P10.16mm_Horizontal
- removed J5: SIM800L_D, TerminalBlock_Phoenix:TerminalBlock_Phoenix_MKDS-3-2-5.08_1x02_P5.08mm_Horizontal
- removed J6: SIM800L_C, TerminalBlock_Phoenix:TerminalBlock_Phoenix_MKDS-3-2-5.08_1x02_P5.08mm_Horizontal
- removed J7: SIM800L_B, TerminalBlock_Phoenix:TerminalBlock_Phoenix_MKDS-3-2-5.08_1x02_P5.08mm_Horizontal
- removed J8: SIM800L_A, TerminalBlock_Phoenix:TerminalBlock_Phoenix_MKDS-3-2-5.08_1x02_P5.08mm_Horizontal
- removed the REF** at (471.5, 157.5)
- removed the REF** at (463.0, 170.0)
- added REF**: OSHW-Logo2_9.8x8mm_SilkScreen, Symbol:OSHW-Logo2_9.8x8mm_SilkScreen, F.Cu at (461.1, 160.5)
- added REF**: KiCad-Logo2_8mm_SilkScreen, Symbol:KiCad-Logo2_8mm_SilkScreen, F.Cu at (477.4, 158.3)
- J9: value POWER -> Power
Routing:
- net +5V: track 504.4 -> 440.6 mm
- net Net-(C3-Pad1): track 20.7 -> 0.00 mm
- net Net-(C4-Pad1): track 20.2 -> 0.00 mm
- net Net-(C1-Pad1): track 19.7 -> 0.00 mm
- net Net-(C2-Pad1): track 13.1 -> 0.00 mm
Other:
- board text added: "SMS Gateway PDU board https://github.com/SniperCZE/sms-gateway"
